Commit message: tugbot simultation for slam and nav

File: src/tugbot_description/urdf/model.urdf.xacro (robot description, xacro)
@@ -3,9 +3,4 @@
   <!-- BASE LINK -->
   <link name="base_link">
-    <inertial>
-      <origin xyz="-0.1 0 0.1" rpy="0 0 0"/>
-      <mass value="46.2"/>
-      <inertia ixx="1.55925" ixy="0" ixz="0" iyy="1.55925" iyz="0" izz="1.55925"/>
-    </inertial>
     <collision name="base_link_collision">
       <origin xyz="0 0 0" rpy="0 0 0"/>
